Commit message: build simple micro mouse with random maze generator

File: src/micro_mouse_description/urdf/mobile_base.xacro (robot description, xacro)
@@ -1,9 +1,14 @@
 <?xml version="1.0"?>
 <robot xmlns:xacro="http://www.ros.org/wiki/xacro">
-    <xacro:property name="base_length" value="0.6"/>
+    <!-- <xacro:property name="base_length" value="0.6"/>
     <xacro:property name="base_width" value="0.4"/>
     <xacro:property name="base_height" value="0.2"/>
     <xacro:property name="wheel_radius" value="0.1"/>
-    <xacro:property name="wheel_length" value="0.05"/>
+    <xacro:property name="wheel_length" value="0.05"/> -->
+    <xacro:property name="base_length" value="0.4"/>
+    <xacro:property name="base_width" value="0.264"/>
+    <xacro:property name="base_height" value="0.132"/>
+    <xacro:property name="wheel_radius" value="0.066"/>
+    <xacro:property name="wheel_length" value="0.033"/>
     <xacro:macro name="wheel_link" params="prefix">
         <link name="${prefix}_wheel_link">

File: src/micro_mouse_description/urdf/mobile_base_gazebo.xacro (robot description, xacro)
@@ -31,5 +31,5 @@
             <odometry_topic>odom</odometry_topic>
             <odometry_frame>odom</odometry_frame>
-            <robot_base_frame>base_footprint</robot_base_frame>
+            <robot_base_frame>base_foot_print</robot_base_frame>
         </plugin>
     </gazebo>
